File: hardware_SI/hardware_SI.sch (KiCad schematic (older format))
At the start: 3 parts, among them U1 OMEGA2+

Commit message: Esq onion power doc v1
Parts:
- added C?: 0.1uF, symbol Device:C
- added C?: 100nF, symbol Device:C
- added D?: LED, symbol Device:LED
- added J?: Conn_02x15_Odd_Even, symbol Connector_Generic:Conn_02x15_Odd_Even
- added R?: 4.99K, symbol Device:R
- added R?: 2M, symbol Device:R
- added R?: 8M, symbol Device:R
- added R?: 330, symbol Device:R
- added SW?: SW_DPDT_x2, symbol Switch:SW_DPDT_x2
- added SW?: SW_MEC_5G, symbol Switch:SW_MEC_5G
- added U?: MCP3021, SOT-23, symbol MCP3021:MCP3021
Connections:
- net +2V5: now also J?.4 (Pin_4), SW?.1 (A), SW?.2 (A)
- net +3V3: now also C?.1, J?.3 (Pin_3), J?.30 (Pin_30), U?.P$1 (VCC)
- net GND: now also C?.2, C?.2, D?.1 (K), J?.1 (Pin_1), J?.26 (Pin_26), J?.29 (Pin_29), R?.2, U?.P$2 (GND)
- net IO0: now also J?.25 (Pin_25)
- net IO1: now also J?.23 (Pin_23)
- net IO12: now also J?.15 (Pin_15)
- net IO13: now also J?.13 (Pin_13)
- net IO14: now also J?.11 (Pin_11)
- net IO18: now also J?.18 (Pin_18)
- net IO19: now also J?.20 (Pin_20)
- net IO20: now also J?.22 (Pin_22), U?.P$5 (SCL)
- net IO21: now also J?.24 (Pin_24), U?.P$4 (SDA)
- net IO23: now also J?.9 (Pin_9)
- net IO26: now also J?.7 (Pin_7)
- net IO6: now also J?.21 (Pin_21)
- net IO7: now also J?.19 (Pin_19)
- net IO8: now also J?.17 (Pin_17)
- net NET_POW: now also J?.5 (Pin_5)
- net RST_B: now also J?.27 (Pin_27)
- net RST_BTN: now also R?.1
- net RX+: now also J?.16 (Pin_16)
- net RX-: now also J?.14 (Pin_14)
- net TX+: now also J?.12 (Pin_12)
- net TX-: now also J?.10 (Pin_10)
- net VCC renamed +BATT
- net +BATT: now also R?.1
- new net: D?.2 (A), R?.2
- new net: R?.2, SW?.3 (B), SW?.4 (B)
- new net +5V: J?.2 (Pin_2), J?.28 (Pin_28), R?.1, SW?.3 (C)
- new net AIN: C?.1, R?.1, R?.2, U?.P$3 (AIN)
- new net D_N: J?.8 (Pin_8)
- new net D_P: J?.6 (Pin_6)
- new net VOUT: SW?.2 (B)
Other:
- moved on the sheet: C?, U?

Commit message: Adelanto en esquemático
Parts:
- added C? (x2): 100n, symbol Device:C
- added C? (x2): 10u, symbol Device:C
- added D? (x3): LED, symbol Device:LED
- added J?: USB_B_Micro, symbol Connector:USB_B_Micro
- added J?: Conn_01x04, symbol Connector_Generic:Conn_01x04
- added R? (x3): 1k, symbol Device:R
- added U? (x2): LD1117S33TR_SOT223, Package_TO_SOT_SMD:SOT-223-3_TabPin2, symbol Regulator_Linear:LD1117S33TR_SOT223
- added U?: MAX6369, Package_TO_SOT_SMD:SOT-23-8, symbol Power_Supervisor:MAX6369
- U1: symbol OMEGA2_:OMEGA2+ -> hardware_SI-rescue:OMEGA2+-OMEGA2_
- U?: symbol INVERTER:INVERTER -> hardware_SI-rescue:INVERTER-INVERTER
- U?: symbol MCP3021:MCP3021 -> hardware_SI-rescue:MCP3021-MCP3021
Connections:
- net GND: now also C?.2, C?.2, C?.2, C?.2, D?.1 (K), D?.1 (K), D?.1 (K), J?.1 (Pin_1), J?.5 (GND), J?.6 (Shield), U?.1 (GND), U?.1 (GND), U?.2 (GND)
- net USB_N: now also J?.2 (D-)
- net USB_P: now also J?.3 (D+)
- new net: D?.2 (A), R?.2 (x3)
- new net Bic_Con: R?.1
- new net Clk_W: U?.1 (WDI)
- new net Lib_Con: R?.1
- new net RST_W: U?.7 (~WDO)
- new net Res_Con: R?.1
- new net SCL: J?.3 (Pin_3)
- new net SDA: J?.4 (Pin_4)
- new net Vcc: J?.2 (Pin_2)
- new net Vin: U?.8 (VCC)
- new net Vin_1: C?.1, J?.1 (VBUS), U?.3 (VI)
- new net Vin_2: C?.1, U?.3 (VI)
- new net Vo_1: C?.1, U?.2 (VO)
- new net Vo_2: C?.1, U?.2 (VO)
- no-connect marks 0 -> 1
