File: hardware_SI/hardware_SI.kicad_sch (KiCad schematic)
At the start: 2 parts, among them U1 OMEGA2+

Commit message: Definiciones PCB
- Se agregan definiciones para la creación de la PCB.
Parts:
- C1: footprint (none) -> Capacitor_SMD:C_0805_2012Metric_Pad1.18x1.45mm_HandSolder
Changed lines of the file:
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@@
       (effects (font (size 1.27 1.27)) (justify left))
     )
-    (property "Footprint" "" (id 2) (at 196.5452 85.09 0)
+    (property "Footprint" "Capacitor_SMD:C_0805_2012Metric_Pad1.18x1.45mm_HandSolder" (id 2) (at 196.5452 85.09 0)
       (effects (font (size 1.27 1.27)) hide)
     )
@@
     )
     (path "/df5c0c0e-e65c-407d-8d2c-4e4d971d84fc"
-      (reference "C1") (unit 1) (value "100n") (footprint "")
+      (reference "C1") (unit 1) (value "100n") (footprint "Capacitor_SMD:C_0805_2012Metric_Pad1.18x1.45mm_HandSolder")
     )
     (path "/d17f886c-ddbc-4da5-b4ad-887fd41c7d7b/79dd93ce-0c87-43fa-8fcb-da2290bc2344"
@@
     )
     (path "/d17f886c-ddbc-4da5-b4ad-887fd41c7d7b/0cf6864d-eb0b-44a4-8430-c2d70446e5de"
-      (reference "C8") (unit 1) (value "100n") (footprint "")
+      (reference "C8") (unit 1) (value "100n") (footprint "Capacitor_SMD:C_0805_2012Metric_Pad1.18x1.45mm_HandSolder")
     )
     (path "/d17f886c-ddbc-4da5-b4ad-887fd41c7d7b/5b4d42a4-f57c-4b7c-a0ea-40675900a8cc"
@@
     )
     (path "/0b6e3c2b-d039-4782-bbc3-fab07ed657e7/fc4f2d85-95e6-494e-ad8e-549d8dc8a347"
-      (reference "C12") (unit 1) (value "100n") (footprint "")
+      (reference "C12") (unit 1) (value "100n") (footprint "Capacitor_SMD:C_0805_2012Metric_Pad1.18x1.45mm_HandSolder")
     )
     (path "/0b6e3c2b-d039-4782-bbc3-fab07ed657e7/05cf4233-8f27-418a-a330-7ad49b161d28"
-      (reference "C13") (unit 1) (value "100n") (footprint "")
+      (reference "C13") (unit 1) (value "100n") (footprint "Capacitor_SMD:C_0805_2012Metric_Pad1.18x1.45mm_HandSolder")
     )
     (path "/5100f047-51fe-4bd1-8576-7ad51d65cc07/a9c7380b-fd51-40e0-9090-6a5b91919810"
@@
     )
     (path "/c5476bbc-f11c-4b73-abe0-40bb556a0d31/8f025fd3-0eaf-44cb-ac32-fb3b91404f49"
-      (reference "R15") (unit 1) (value "1k") (footprint "")
+      (reference "R15") (unit 1) (value "1k") (footprint "Resistor_SMD:R_0805_2012Metric_Pad1.20x1.40mm_HandSolder")
     )
     (path "/c5476bbc-f11c-4b73-abe0-40bb556a0d31/46dc8b71-656c-468b-90ed-7b333fd4b86b"
-      (reference "R16") (unit 1) (value "1k") (footprint "")
+      (reference "R16") (unit 1) (value "1k") (footprint "Resistor_SMD:R_0805_2012Metric_Pad1.20x1.40mm_HandSolder")
     )
     (path "/d17f886c-ddbc-4da5-b4ad-887fd41c7d7b/ab8397f0-cb8b-42a3-97b6-8f2bb790bc88"
@@
     )
     (path "/5100f047-51fe-4bd1-8576-7ad51d65cc07/c3617d4b-43cd-435a-a463-91a105f5bb7d"
-      (reference "U6") (unit 1) (value "MCP3021") (footprint "SOT95P270X145-5N")
+      (reference "U6") (unit 1) (value "MCP3021") (footprint "MCP3021A5T-E_OT:SOT95P270X145-5N")
     )
     (path "/c5476bbc-f11c-4b73-abe0-40bb556a0d31/f1b1be8e-77a3-403b-a3de-1117b066b8c9"
