File: hardware_SI/hardware_SI.kicad_pcb (KiCad board)
At the start: 2 copper layers, 228 x 147.6 mm, 58 parts, among them J1 Barrel_Jack_Switch, J2 Conn_01x07_Female, J3 USB_B_Micro, Q1 SI2323DS-T1, Q2 SI2323DS-T1, SW1 SW_SPDT, U1 OMEGA2+, U2 LTC4085EDEPBF, U3 TPS61200DRC, U4 LD1117S33TR_SOT223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

Commit message: adding branch dev_dch
Parts:
- BT1: moved to B.Cu
- moved R16 153.2 mm to (210.8, 157.5)
- moved R15 150.6 mm to (213.4, 152.4)
- moved R14 147.7 mm to (35.6, 144.8)
- moved C18 144.3 mm to (210.8, 144.8)
- moved U8 136.6 mm to (195.6, 149.9), turned to 180 degrees
- moved C17 133.6 mm to (200.7, 157.5)
- moved C1 133.6 mm to (213.4, 35.6)
- moved TH1 120.3 mm to (216.8, 88.9)
- moved C13 107.4 mm to (144.8, 78.7), turned to 90 degrees
- moved C15 100.6 mm to (94.0, 127.0), turned to -90 degrees
- moved J2 97.1 mm to (149.9, 76.2)
- moved D3 90.8 mm to (246.4, 109.2)
- moved J3 90.4 mm to (147.3, 144.8)
- moved D2 89.8 mm to (248.9, 94.0)
- moved R1 88.4 mm to (248.9, 101.6)
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
Commit message: PCB V1
Parts:
- moved SW1 167.9 mm to (248.9, 83.8), turned to 90 degrees
- moved FB1 156.0 mm to (241.3, 27.9), turned to 180 degrees
- moved J3 152.9 mm to (248.9, 30.5), turned to 90 degrees
- moved U4 151.0 mm to (238.8, 83.8)
- moved C16 150.9 mm to (228.6, 30.5)
- moved C10 149.9 mm to (231.1, 86.4), turned to 90 degrees
- moved C11 141.2 mm to (231.1, 81.3), turned to 90 degrees
- moved C14 136.8 mm to (152.4, 68.6)
- moved R14 136.8 mm to (152.4, 73.7)
- moved R13 132.5 mm to (157.5, 71.1)
- moved C17 131.9 mm to (236.2, 30.5), turned to 90 degrees
- moved U7 131.4 mm to (245.2, 39.0)
- moved D3 123.8 mm to (134.6, 55.9)
- moved U8 118.9 mm to (236.2, 38.1)
- moved C4 118.2 mm to (137.2, 50.8)
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
Commit message: PCB V2
Parts:
- moved R2 94.3 mm to (217.4, 81.3), turned to 180 degrees
- moved C8 90.6 mm to (206.4, 83.2)
- moved Q2 88.7 mm to (216.1, 71.4)
- moved R5 83.9 mm to (199.1, 71.8), turned to 180 degrees
- moved C3 82.8 mm to (215.9, 76.8)
- moved R6 78.2 mm to (195.9, 80.6), turned to 180 degrees
- moved TH1 78.1 mm to (195.9, 74.9)
- moved U2 77.9 mm to (205.7, 76.8), turned to 180 degrees
- moved C14 76.9 mm to (227.3, 51.4), turned to 180 degrees
- moved R14 76.5 mm to (227.0, 56.5), turned to 180 degrees
- moved C2 75.6 mm to (210.6, 83.2)
- moved R13 69.9 mm to (226.7, 61.6)
- moved C5 67.9 mm to (206.1, 71.1), turned to 180 degrees
- moved C15 59.8 mm to (226.9, 46.4), turned to 180 degrees
- moved Q1 59.7 mm to (186.7, 80.0), turned to -90 degrees
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Routing:
- net +3V3: track 0.00 -> 190.8 mm, vias 0 -> 2
- net +5VA: track 0.00 -> 144.9 mm
- net +5VL: track 0.00 -> 143.2 mm, vias 0 -> 2
- net +5VP: track 0.00 -> 105.6 mm, vias 0 -> 2
- net +BATT: track 0.00 -> 97.3 mm, vias 0 -> 3
- net /WDI: track 0.00 -> 52.1 mm, vias 0 -> 1
- net /sistema_alimentacion/*ACPR: track 0.00 -> 45.7 mm
- net /IO19: track 0.00 -> 40.5 mm
- net Net-(C7-Pad1): track 0.00 -> 29.8 mm
- net Net-(Q2-Pad1): track 0.00 -> 29.5 mm, vias 0 -> 3
- net Net-(J3-Pad2): track 0.00 -> 29.1 mm, vias 0 -> 1
- net /RST_W: track 0.00 -> 28.7 mm
- net /CS1: track 0.00 -> 27.5 mm
- net Net-(J3-Pad3): track 0.00 -> 26.2 mm
- net Net-(C6-Pad1): track 0.00 -> 23.6 mm
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- added copper zone on F.Cu, net GND
- added copper zone on F.Cu, net GNDPWR
Other:
- board size 228 x 147.6 mm -> 96.6 x 81.6 mm
