File: hardware_SI/programacion.kicad_sch (KiCad schematic)
At the start: 9 parts, among them J3 USB_B_Micro, U7 USBLC6-2SC6, U8 CH340N

Commit message: Definiciones PCB
- Se agregan definiciones para la creación de la PCB.
Parts:
- R15, R16: footprint (none) -> Resistor_SMD:R_0805_2012Metric_Pad1.20x1.40mm_HandSolder
Changed lines of the file:
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@@
     (property "Reference" "R16" (id 0) (at 199.39 83.82 90))
     (property "Value" "1k" (id 1) (at 199.39 81.28 90))
-    (property "Footprint" "" (id 2) (at 199.39 79.502 90)
+    (property "Footprint" "Resistor_SMD:R_0805_2012Metric_Pad1.20x1.40mm_HandSolder" (id 2) (at 199.39 79.502 90)
       (effects (font (size 1.27 1.27)) hide)
     )
@@
     (property "Reference" "R15" (id 0) (at 199.39 76.2 90))
     (property "Value" "1k" (id 1) (at 199.39 78.74 90))
-    (property "Footprint" "" (id 2) (at 199.39 76.962 90)
+    (property "Footprint" "Resistor_SMD:R_0805_2012Metric_Pad1.20x1.40mm_HandSolder" (id 2) (at 199.39 76.962 90)
       (effects (font (size 1.27 1.27)) hide)
     )
